File: Sendor_Board.sch (EAGLE design)
At the start: 54 parts, among them Q1 8.000Mhz, T1 IRLM6402TRPBF, U1 PIC32MX795F512H-80I/PT, U2 SHT25, U3 MPL115A2, U4 MRF24J40MA, U5 TC1262-3.3VDB, U6 VTX-214-003-105, X1 MINI-USB-SHIELD-UX60A-MB-5ST, X2 MSTBA4

Commit message: Some correction
Parts:
- CONF, CONF-1°C, CONF-2°C, ECO, POWER: value (none) -> KPT-2012YC
- F1: value (none) -> 0031.8201
- PROG: value (none) -> 826926-6
- S1: value (none) -> B3F-3100
Changed lines of the file:
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@@
 <part name="GND13" library="supply1" deviceset="GND" device=""/>
 <part name="GND14" library="supply1" deviceset="GND" device=""/>
-<part name="F1" library="fuse" deviceset="SH22,5" device=""/>
+<part name="F1" library="fuse" deviceset="SH22,5" device="" value="0031.8201"/>
 <part name="D1" library="diode" deviceset="1N4004" device=""/>
 <part name="D2" library="diode" deviceset="1N4004" device=""/>
@@
 <part name="T1" library="zetex" deviceset="PMOSSOT23" device="" value="IRLM6402TRPBF"/>
 <part name="D3" library="diode" deviceset="DIODE-" device="DO214AC" value="B340A-E3/61T"/>
-<part name="PROG" library="con-lstb" deviceset="MA06-1" device=""/>
+<part name="PROG" library="con-lstb" deviceset="MA06-1" device="" value="826926-6"/>
 <part name="GND18" library="supply1" deviceset="GND" device=""/>
 <part name="+3V7" library="supply1" deviceset="+3V3" device=""/>
 <part name="+3V8" library="supply1" deviceset="+3V3" device=""/>
-<part name="CONF" library="led" deviceset="LED" device="CHIP-LED0805"/>
-<part name="CONF-1°C" library="led" deviceset="LED" device="CHIP-LED0805"/>
-<part name="POWER" library="led" deviceset="LED" device="CHIP-LED0805"/>
-<part name="ECO" library="led" deviceset="LED" device="CHIP-LED0805"/>
-<part name="CONF-2°C" library="led" deviceset="LED" device="CHIP-LED0805"/>
+<part name="CONF" library="led" deviceset="LED" device="CHIP-LED0805" value="KPT-2012YC"/>
+<part name="CONF-1°C" library="led" deviceset="LED" device="CHIP-LED0805" value="KPT-2012YC"/>
+<part name="POWER" library="led" deviceset="LED" device="CHIP-LED0805" value="KPT-2012YC"/>
+<part name="ECO" library="led" deviceset="LED" device="CHIP-LED0805" value="KPT-2012YC"/>
+<part name="CONF-2°C" library="led" deviceset="LED" device="CHIP-LED0805" value="KPT-2012YC"/>
 <part name="R8" library="resistor" deviceset="R-EU_" device="R1206" value="1K"/>
 <part name="R9" library="resistor" deviceset="R-EU_" device="R1206" value="1K"/>
@@
 <part name="R11" library="resistor" deviceset="R-EU_" device="R1206" value="1K"/>
 <part name="R12" library="resistor" deviceset="R-EU_" device="R1206" value="1K"/>
-<part name="S1" library="switch-omron" deviceset="31-XX" device=""/>
+<part name="S1" library="switch-omron" deviceset="31-XX" device="" value="B3F-3100"/>
 <part name="R13" library="resistor" deviceset="R-EU_" device="R1206" value="1k"/>
 <part name="+3V9" library="supply1" deviceset="+3V3" device=""/>
@@
 <wire x1="200.66" y1="86.36" x2="190.5" y2="86.36" width="0.1524" layer="91"/>
 <wire x1="190.5" y1="86.36" x2="190.5" y2="88.9" width="0.1524" layer="91"/>
+<junction x="220.98" y="86.36"/>
+<junction x="210.82" y="86.36"/>
+<junction x="200.66" y="86.36"/>
 </segment>
 <segment>
@@
 <wire x1="200.66" y1="99.06" x2="190.5" y2="99.06" width="0.1524" layer="91"/>
 <wire x1="190.5" y1="99.06" x2="190.5" y2="96.52" width="0.1524" layer="91"/>
+<junction x="200.66" y="99.06"/>
+<junction x="210.82" y="99.06"/>
+<junction x="220.98" y="99.06"/>
 </segment>
 <segment>
@@
 <wire x1="198.12" y1="27.94" x2="205.74" y2="27.94" width="0.1524" layer="91"/>
 <pinref part="U1" gate="A" pin="OSC2/CLKO/RC15"/>
+<junction x="198.12" y="27.94"/>
 </segment>
 </net>
@@
 <wire x1="198.12" y1="12.7" x2="205.74" y2="12.7" width="0.1524" layer="91"/>
 <pinref part="U1" gate="A" pin="OSC1/CLKI/RC12"/>
+<junction x="198.12" y="12.7"/>
 </segment>
 </net>
@@
 <wire x1="149.86" y1="-38.1" x2="149.86" y2="-40.64" width="0.1524" layer="91"/>
 <junction x="177.8" y="-33.02"/>
-</segment>
-</net>
+<junction x="162.56" y="-33.02"/>
+</segment>
+</net>
