File: CaptorBoard.sch (KiCad schematic (older format))
At the start: 55 parts, among them CON1 MINI-USB-SHELD-MC32598, P1 Prog, P2 POWER, P3 EXT, Q1 IRLM6402TRPBF, SW1 SKHHLVA010, U1 PIC32MX795F512H-80I-PT, U2 MRF24J40MA-I-RM, U3 SHT25, U4 MPL115A2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

Commit message: finally use WeMos Mini
Parts:
- removed C1, C10, C11, C12, C13, C15, C3, C4, C8, C9: 100nF, Capacitors_SMD:C_0805, symbol C
- removed C14: 1uF, Capacitors_SMD:C_0805, symbol C
- removed C16: 1uF, Capacitors_SMD:c_elec_4x5.3, symbol CP
- removed C2: 10uF, Capacitors_SMD:c_elec_5x5.3, symbol CP
- removed C5: TPSA106K010R0900, SMD_Packages:SMD-1206_Pol, symbol CP
- removed C6, C7: 20pF, Capacitors_SMD:C_0805, symbol C
- removed CON1: MINI-USB-SHELD-MC32598, pfo:USB_Mini-B, symbol USB-MINI-B
- removed D1, D2: BAS32L, Diodes_SMD:Diode-MiniMELF_Standard, symbol D_Small
- removed D8: B340A-E3/61T, Diodes_SMD:Diode-SMB_Standard, symbol D
- removed F1: F_Small, Fuse_Holders_and_Fuses:Fuseholder5x20_horiz_SemiClosed_Casing10x25mm, symbol F_Small
- removed P1: Prog, Pin_Headers:Pin_Header_Straight_1x06, symbol CONN_01X06
- removed P2: POWER, Connect:bornier4, symbol CONN_01X04
- removed P3: EXT, Pin_Headers:Pin_Header_Straight_1x04, symbol CONN_01X04
- removed Q1: IRLM6402TRPBF, Housings_SOT-23_SOT-143_TSOT-6:SOT-23, symbol IRLM6402TRPBF
- removed R1: 68k, Resistors_SMD:R_0805, symbol R
- removed R2, R6: 1k, Resistors_SMD:R_0805, symbol R
- removed R3: 10R, Resistors_SMD:R_0805, symbol R
- removed R4, R5: 2.2k, Resistors_SMD:R_0805, symbol R
- removed U1: PIC32MX795F512H-80I-PT, Housings_QFP:TQFP-64_10x10mm_Pitch0.5mm, symbol PIC32MX795F512H-80I-PT
- removed U2: MRF24J40MA-I-RM, pfo:MRF24J40MA, symbol MRF24J40MA-I-RM
- removed U3: SHT25, pfo:HTU21, symbol HTU21
- removed U4: MPL115A2, pfo:MPL115A2, symbol MPL115A2
- removed U5: VTX-214-005-005, pfo:VTX-214-005-x, symbol VTX-214-003-105
- removed U6: TC1262-3.3VDB, SMD_Packages:SOT-223, symbol TC1262-3.3VDB
- removed U7, U8: MOC3042M, Housings_DIP:DIP-6__300_ELL, symbol MOC3042M
- removed Y1: FQ7050B-8.000, pfo:SMD_Crystal_FQ7050_Series, symbol Crystal_Small
- added J1: Conn_01x06, Pin_Headers:Pin_Header_Straight_1x06_Pitch2.54mm, symbol Connector:Conn_01x06
- added J2: Screw_Terminal_01x04, Connectors_Terminal_Blocks:TerminalBlock_bornier-4_P5.08mm, symbol CaptorBoard-rescue:Screw_Terminal_01x04
- added SW2: SKHHLVA010, Buttons_Switches_THT:SW_Tactile_SKHH_Angled, symbol CaptorBoard-rescue:SW_PUSH
- added U1: WeMos_mini, wemos-d1-mini:wemos-d1-mini-with-pin-header-and-connector, symbol wemos_mini:WeMos_mini
- added U2: IRM-02-5, Converters_DCDC_ACDC:ACDC-Conv_THTMeanWell-IRM-02-XX, symbol pfo:IRM-02-5
- added U3, U4: MOC3041M, Housings_DIP:DIP-6_W7.62mm, symbol opto:MOC3041M
- added U5: DHT22, pfo:DHT22_Temperature_Humidity, symbol pfo:DHT22
- D10, D9: footprint Diodes_ThroughHole:Diode_DO-41_SOD81_Horizontal_RM10 -> Diodes_THT:D_DO-41_SOD81_P7.62mm_Horizontal; symbol D -> CaptorBoard-rescue:D-RESCUE-CaptorBoard
- D3, D4, D5, D6, D7: footprint LEDs:LED-3MM -> LEDs:LED_D3.0mm_Horizontal_O1.27mm_Z2.0mm; symbol LED -> CaptorBoard-rescue:LED-RESCUE-CaptorBoard
- R10, R11, R7, R8, R9: footprint Resistors_SMD:R_0805 -> Resistors_SMD:R_1210_HandSoldering; symbol R -> device:R
- R12, R13: footprint Resistors_SMD:R_0805 -> Resistors_SMD:R_2010_HandSoldering; symbol R -> device:R
- SW1: footprint pfo:CST06S -> Buttons_Switches_THT:SW_Tactile_SKHH_Angled; symbol SW_PUSH -> CaptorBoard-rescue:SW_PUSH
Connections:
- net labels added: ANA, CAPTOR, RESET
- net labels removed: *MCLR, 5V_SEC, CS_RF, D+, D-, INT_RF, PGC, PGD, Phase_F, RST_PRES, RST_RF, SCK_RF, SCL_CAP, SDA_CAP, SDI_RF, SDO_RF, SHD_PRES, USBID, VUSB, WK_RF
- wire segments 219 -> 91
- no-connect marks 24 -> 1
Other:
- note added: "CPU"
- note removed: "Humidity and \ntemperatuer sensor\n"
- note removed: "Pressure sensor"
- note removed: "Radio transmission"
- moved on the sheet: SW1

Commit message: Board final
Parts:
- added F1: Fuse_Small, Fuse:Fuseholder_Littelfuse_Nano2_157x, symbol device:Fuse_Small
- D3, D4, D5, D6, D7: footprint LEDs:LED_D3.0mm_Horizontal_O1.27mm_Z2.0mm -> LEDs:LED_D3.0mm
- J1: symbol Connector:Conn_01x06 -> CaptorBoard-rescue:Conn_01x06-Connector
- J2: value Screw_Terminal_01x04 -> MKDSN 1,5/ 4-5,08; footprint Connectors_Terminal_Blocks:TerminalBlock_bornier-4_P5.08mm -> TerminalBlocks_Phoenix:TerminalBlock_Phoenix_MKDS1.5-4pol
- R10, R11, R7, R8, R9: symbol device:R -> CaptorBoard-rescue:R-device
- R12, R13: footprint Resistors_SMD:R_2010_HandSoldering -> Resistors_SMD:R_1210_HandSoldering; symbol device:R -> CaptorBoard-rescue:R-device
- U3, U4: value MOC3041M -> MOC3040X; symbol opto:MOC3041M -> CaptorBoard-rescue:MOC3041M-opto
Connections:
- net labels added: CMD1, CMD2
- net labels removed: Pilote, Terre
- wire segments 91 -> 92
Other:
- moved on the sheet: D3, D4, D5, D6, D7, J2, R10, R11, R7, R8, R9, U2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
