File: CaptorBoard.kicad_sch (KiCad schematic)
At the start: 50 parts, among them J1 Conn_01x06, J2 Screw_Terminal_01x03, J3 Screw_Terminal_01x03, J4 Conn_01x07, J5 Conn_01x04, J6 Screw_Terminal_01x03, K1 G5LE-1-DC5, K2 G5LE-1-DC5, Q1 2N7002E, Q2 2N7002E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

Commit message: Add open source hardware logo
Parts:
- added LOGO1: Logo_Open_Hardware_Large, Symbol:OSHW-Logo_11.4x12mm_SilkScreen, symbol Graphic:Logo_Open_Hardware_Large
Changed lines of the file:
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@@
     (pin "5")
+  )
+  (symbol (lib_id "Graphic:Logo_Open_Hardware_Large") (at 387.35 123.19 0) (unit 1)
+    (in_bom no) (on_board yes) (fields_autoplaced)
+    (property "Reference" "LOGO1" (id 0) (at 387.35 110.49 0)
+      (effects (font (size 1.27 1.27)) hide)
+    )
+    (property "Value" "Logo_Open_Hardware_Large" (id 1) (at 387.35 133.35 0)
+      (effects (font (size 1.27 1.27)) hide)
+    )
+    (property "Footprint" "Symbol:OSHW-Logo_11.4x12mm_SilkScreen" (id 2) (at 387.35 123.19 0)
+      (effects (font (size 1.27 1.27)) hide)
+    )
+    (property "Datasheet" "~" (id 3) (at 387.35 123.19 0)
+      (effects (font (size 1.27 1.27)) hide)
+    )
   )
   (symbol (lib_id "Device:Crystal") (at 44.45 95.25 90) (unit 1)
@@
       (reference "K2") (unit 1) (value "G5LE-1-DC5") (footprint "Relay_THT:Relay_SPDT_Omron-G5LE-1")
     )
+    (path "/9ce2f92b-9802-4b50-84da-c9575dee9722"
+      (reference "LOGO1") (unit 1) (value "Logo_Open_Hardware_Large") (footprint "Symbol:OSHW-Logo_11.4x12mm_SilkScreen")
+    )
     (path "/43b55e6c-f551-41f8-baf6-d6b8e6806cfa"

Commit message: Change relait and LED schematic
Parts:
- removed D11, D2: MRA4007T3G, Diode_SMD:D_SMA, symbol Diode:MRA4007T3G
- added D11, D2: 1N4148W, Diode_SMD:D_SOD-123, symbol Diode:1N4148W
- R4, R6: value 1k -> 10k
Connections:
- net +5V: now also D11.1 (K), D2.1 (K); no longer R14.1, R5.1
- net GND: now also D1.1 (K), D8.1 (K), R4.2, R6.2
- net REL1: now also Q1.1 (G), R4.1, R5.1; no longer R4.2
- net REL2: now also Q2.1 (G), R14.1, R6.1; no longer R6.2
- net at K2.2, Q2.3 (D): now also D11.2 (A); no longer D8.1 (K)
- net at K1.2, Q1.3 (D): now also D2.2 (A); no longer D1.1 (K)
Other:
- moved on the sheet: C1, C6, D1, D10, D3, D4, D5, D6, D7, D8, D9, K1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
